Commit message: pico Dshot publisher and gamepad based controller

File: src/hydrogen/model/propellers.xacro (robot description, xacro)
@@ -75,5 +75,5 @@
       izz="0.0008"/>
     <!-- Joints -->
-    <joint name="front_propeller_joint" type="continuous">
+    <joint name="back_propeller_joint" type="continuous">
       <parent link="hydrogen_frame"/>
       <child link="front_propeller"/>
@@ -81,5 +81,5 @@
       <axis xyz="0 0 1"/>
     </joint>
-    <joint name="left_propeller_1_joint" type="continuous">
+    <joint name="right_propeller_1_joint" type="continuous">
       <parent link="hydrogen_frame"/>
       <child link="left_propeller_1"/>
@@ -87,5 +87,5 @@
       <axis xyz="0 0 1"/>
     </joint>
-    <joint name="left_propeller_2_joint" type="continuous">
+    <joint name="right_propeller_2_joint" type="continuous">
       <parent link="hydrogen_frame"/>
       <child link="left_propeller_2"/>
@@ -93,5 +93,5 @@
       <axis xyz="0 0 1"/>
     </joint>
-    <joint name="right_propeller_1_joint" type="continuous">
+    <joint name="left_propeller_1_joint" type="continuous">
       <parent link="hydrogen_frame"/>
       <child link="right_propeller_1"/>
@@ -99,5 +99,5 @@
       <axis xyz="0 0 1"/>
     </joint>
-    <joint name="right_propeller_2_joint" type="continuous">
+    <joint name="left_propeller_2_joint" type="continuous">
       <parent link="hydrogen_frame"/>
       <child link="right_propeller_2"/>
