Commit message: Rtab_map

File: src/hydrogen/model/cameras.xacro (robot description, xacro)
@@ -6,5 +6,5 @@
       <visual>
         <geometry>
-          <mesh filename="package://hydrogen/meshes/zed2i.stl"/>
+          <mesh filename="file://$(find hydrogen)/meshes/zed2i.stl"/>
         </geometry>
         <material name="zed_mat">
@@ -14,5 +14,5 @@
       <collision>
         <geometry>
-          <mesh filename="package://hydrogen/meshes/zed2i.stl"/>
+          <mesh filename="file://$(find hydrogen)/meshes/zed2i.stl"/>
         </geometry>
       </collision>
@@ -44,6 +44,6 @@
           <horizontal_fov>1.92</horizontal_fov>
           <image>
-            <width>1280</width>
-            <height>720</height>
+            <width>800</width>
+            <height>600</height>
             <format>R8G8B8</format>
           </image>

File: src/hydrogen/model/main_frame.xacro (robot description, xacro)
@@ -18,5 +18,5 @@
         <geometry>
           <mesh
-            filename="package://hydrogen/meshes/auv2.stl"
+            filename="file://$(find hydrogen)/meshes/auv2.stl"
             scale="0.001 0.001 0.001"/>
         </geometry>

File: src/hydrogen/model/propellers.xacro (robot description, xacro)
@@ -17,5 +17,5 @@
         <geometry>
           <mesh
-            filename="package://hydrogen/meshes/${mesh}"
+            filename="file://$(find hydrogen)/meshes/${mesh}"
             scale="${scale}"/>
         </geometry>
@@ -27,5 +27,5 @@
         <geometry>
           <mesh
-            filename="package://hydrogen/meshes/${mesh}"
+            filename="file://$(find hydrogen)/meshes/${mesh}"
             scale="${scale}"/>
         </geometry>

Commit message: rtabmap_transform fix

File: src/hydrogen/model/cameras.xacro (robot description, xacro)
@@ -3,4 +3,5 @@
   <!-- ================= ZED CAMERA MACRO ================= -->
   <xacro:macro name="zed_camera" params="name parent xyz rpy">
+    <!-- ================= Camera Physical Link ================= -->
     <link name="${name}">
       <visual>
@@ -28,4 +29,5 @@
       </inertial>
     </link>
+    <!-- Mount camera to parent -->
     <joint name="${name}_joint" type="fixed">
       <parent link="${parent}"/>
@@ -33,5 +35,14 @@
       <origin xyz="${xyz}" rpy="${rpy}"/>
     </joint>
-    <!-- Gazebo RGBD camera -->
+    <!-- ================= Optical Frame (CRITICAL FIX) ================= -->
+    <!-- Converts robot frame (X forward, Z up)
+         to optical frame (Z forward, X right, Y down) -->
+    <link name="${name}_optical_frame"/>
+    <joint name="${name}_optical_joint" type="fixed">
+      <parent link="${name}"/>
+      <child link="${name}_optical_frame"/>
+      <origin xyz="0 0 0" rpy="-1.5708 0 -1.5708"/>
+    </joint>
+    <!-- ================= Gazebo RGBD Camera ================= -->
     <gazebo reference="${name}">
       <sensor name="${name}_sensor" type="rgbd_camera">
@@ -39,5 +50,6 @@
         <update_rate>30</update_rate>
         <visualize>true</visualize>
-        <ignition_frame_id>${name}</ignition_frame_id>
+        <!-- IMPORTANT: Publish images in optical frame -->
+        <ignition_frame_id>${name}_optical_frame</ignition_frame_id>
         <topic>${name}</topic>
         <camera>
