Commit message: uart logger

File: src/hydrogen/model/main_frame.xacro (robot description, xacro)
@@ -6,5 +6,5 @@
       <inertial>
         <origin xyz="0.0 0.0 -0.25" rpy="0 0 0"/>
-        <mass value="40.0"/>
+        <mass value="45.0"/>
         <inertia
           ixx="0.2276"

Commit message: Deuterium stl changes

File: src/hydrogen/model/main_frame.xacro (robot description, xacro)
@@ -5,6 +5,6 @@
     <link name="hydrogen_frame">
       <inertial>
-        <origin xyz="0.0 0.0 -0.25" rpy="0 0 0"/>
-        <mass value="45.0"/>
+        <origin xyz="0.0 0.0 -0.25" rpy="0 0 -1.57"/>
+        <mass value="12.0"/>
         <inertia
           ixx="0.2276"
@@ -16,7 +16,8 @@
       </inertial>
       <visual>
+      <origin xyz="0.008 0.0 0.0" rpy="0 0 1.57"/>
         <geometry>
           <mesh
-            filename="file://$(find hydrogen)/meshes/auv2.stl"
+            filename="file://$(find hydrogen)/meshes/auv.stl"
             scale="0.001 0.001 0.001"/>
         </geometry>
@@ -26,5 +27,5 @@
       </visual>
       <collision name="hydrogen_frame_collision">
-        <origin xyz="0.008 0.0 0.0" rpy="0 0 0"/>
+        <origin xyz="0.008 0.0 0.0" rpy="0 0 -1.57"/>
         <geometry>
           <box size="0.45 0.45 0.25"/>

File: src/hydrogen/model/propellers.xacro (robot description, xacro)
@@ -78,5 +78,5 @@
       <parent link="hydrogen_frame"/>
       <child link="front_propeller"/>
-      <origin xyz="-0.223 -0.00725 0.002" rpy="0 0 0"/>
+      <origin xyz="-0.3219 -0 0.0775" rpy="0 0 0"/>
       <axis xyz="0 0 1"/>
     </joint>
@@ -84,5 +84,5 @@
       <parent link="hydrogen_frame"/>
       <child link="left_propeller_1"/>
-      <origin xyz="-0.0631 -0.1734 0.016" rpy="-1.57 0 1.57"/>
+      <origin xyz="-0.1532 0.222 0.085" rpy="-1.57 0 1.57"/>
       <axis xyz="0 0 1"/>
     </joint>
@@ -90,5 +90,5 @@
       <parent link="hydrogen_frame"/>
       <child link="left_propeller_2"/>
-      <origin xyz="0.0697 -0.1734 0.002" rpy="0 0 0"/>
+      <origin xyz="0.1737 0.222 0.0775" rpy="0 0 0"/>
       <axis xyz="0 0 1"/>
     </joint>
@@ -96,5 +96,5 @@
       <parent link="hydrogen_frame"/>
       <child link="right_propeller_1"/>
-      <origin xyz="-0.0631 0.1734 0.016" rpy="-1.57 0 1.57"/>
+      <origin xyz="-0.1532 -0.222 0.085" rpy="-1.57 0 1.57"/>
       <axis xyz="0 0 1"/>
     </joint>
@@ -102,5 +102,5 @@
       <parent link="hydrogen_frame"/>
       <child link="right_propeller_2"/>
-      <origin xyz="0.0697 0.1734 0.002" rpy="0 0 0"/>
+      <origin xyz="00.1737 -0.222 0.0775" rpy="0 0 0"/>
       <axis xyz="0 0 1"/>
     </joint>

File: src/hydrogen/model/robot.xacro (robot description, xacro)
@@ -10,10 +10,10 @@
     name="zed_camera_front_link"
     parent="hydrogen_frame"
-    xyz="0.162 0 0.016"
+    xyz="0.31 0 0.1"
     rpy="0 0 0"/>
   <xacro:zed_camera
     name="zed_camera_down_link"
     parent="hydrogen_frame"
-    xyz="0.05 0 -0.08"
+    xyz="0.17 0 -0.04"
     rpy="0 1.5708 0"/>
 </robot>

Commit message: Inertia corrected for Deuterium

File: src/hydrogen/model/main_frame.xacro (robot description, xacro)
@@ -5,13 +5,7 @@
     <link name="hydrogen_frame">
       <inertial>
-        <origin xyz="0.0 0.0 -0.25" rpy="0 0 -1.57"/>
+        <origin xyz="0.0 0.0 0.0" rpy="0 0 0"/>
         <mass value="12.0"/>
-        <inertia
-          ixx="0.2276"
-          ixy="-0.004544"
-          ixz="-0.0004496"
-          iyy="0.1921"
-          iyz="-0.0001196"
-          izz="0.3559"/>
+<inertia ixx="0.391803" iyy="0.876695" izz="1.065444" ixy="0.0" iyz="0.0" ixz="-0.006759"/>
       </inertial>
       <visual>
@@ -27,7 +21,7 @@
       </visual>
       <collision name="hydrogen_frame_collision">
-        <origin xyz="0.008 0.0 0.0" rpy="0 0 -1.57"/>
+        <origin xyz="0.0 0.0 0.1" rpy="0 0 0"/>
         <geometry>
-          <box size="0.45 0.45 0.25"/>
+          <box size="0.75 0.55 0.3"/>
         </geometry>
       </collision>

Commit message: fixed innertia and added RTABmap

File: src/hydrogen/model/main_frame.xacro (robot description, xacro)
@@ -6,6 +6,12 @@
       <inertial>
         <origin xyz="0.0 0.0 0.0" rpy="0 0 0"/>
-        <mass value="12.0"/>
-<inertia ixx="0.391803" iyy="0.876695" izz="1.065444" ixy="0.0" iyz="0.0" ixz="-0.006759"/>
+        <mass value="45.0"/>
+        <inertia
+          ixx="0.2276"
+          ixy="-0.004544"
+          ixz="-0.0004496"
+          iyy="0.1921"
+          iyz="-0.0001196"
+          izz="0.3559"/>
       </inertial>
       <visual>
@@ -21,5 +27,5 @@
       </visual>
       <collision name="hydrogen_frame_collision">
-        <origin xyz="0.0 0.0 0.1" rpy="0 0 0"/>
+        <origin xyz="-0.00013 0.0 0.15" rpy="0 0 0"/>
         <geometry>
           <box size="0.75 0.55 0.3"/>

Commit message: rtabmap_fix

File: src/hydrogen/model/main_frame.xacro (robot description, xacro)
@@ -6,5 +6,5 @@
       <inertial>
         <origin xyz="0.0 0.0 0.0" rpy="0 0 0"/>
-        <mass value="45.0"/>
+        <mass value="50.0"/>
         <inertia
           ixx="0.2276"

Commit message: PID tuning

File: src/hydrogen/model/main_frame.xacro (robot description, xacro)
@@ -6,5 +6,5 @@
       <inertial>
         <origin xyz="0.0 0.0 0.0" rpy="0 0 0"/>
-        <mass value="50.0"/>
+        <mass value="45.0"/>
         <inertia
           ixx="0.2276"

Commit message: added pico_controller and fixed Buoyancy

File: src/hydrogen/model/main_frame.xacro (robot description, xacro)
@@ -6,12 +6,12 @@
       <inertial>
         <origin xyz="0.0 0.0 0.0" rpy="0 0 0"/>
-        <mass value="45.0"/>
+        <mass value="33.93"/>
         <inertia
-          ixx="0.2276"
-          ixy="-0.004544"
-          ixz="-0.0004496"
-          iyy="0.1921"
-          iyz="-0.0001196"
-          izz="0.3559"/>
+          ixx="0.1716"
+          ixy="-0.003426"
+          ixz="-0.0003390"
+          iyy="0.1448"
+          iyz="-0.00009018"
+          izz="0.2683"/>
       </inertial>
       <visual>
@@ -27,7 +27,7 @@
       </visual>
       <collision name="hydrogen_frame_collision">
-        <origin xyz="-0.00013 0.0 0.15" rpy="0 0 0"/>
+        <origin xyz="-0.00013 0.0 0.12" rpy="0 0 0"/>
         <geometry>
-          <box size="0.75 0.55 0.3"/>
+          <box size="0.45 0.35 0.22"/>
         </geometry>
       </collision>
